File: KiCAD/Four Channel MHz LED Driver/Four Channel MHz LED Driver.sch (KiCad schematic (older format))
At the start: 75 parts, among them J1 Barrel_Jack_Switch, J2 Conn_01x02_Female, J3 8P8C_Shielded_x4, J5 Conn_01x24_Female, J6 Conn_01x05_Male, J7 Conn_01x24_Female, J9 Conn_01x04_Male, M1 Fan_4pin, Q2 SUM70060E, SW1 G13JVCF, U1 S20V18F122V_DC, U10 LT6200CS8-10, U14 Teensy3.6, U16 SN74LV4T125PWR, U2 ASSR-1218, U3 DPBW06F-05, U4 BDJ0GA5WEFJ-E2, U5 ADP7182AUJZ-1.8-R7, U6 TMUX1204DGSR, U7 ASSR-1218, U8 ASSR-1218, U9 ASSR-1218

Commit message: Starting layout
Parts:
- removed C11: 47uF, Capacitor_SMD:C_1206_3216Metric, symbol Device:C_Small
- removed C4: 14000uF, Capacitor_SMD:CP_Elec_18x22, symbol Device:CP1_Small
- removed D3: D_Zener_x4_ACom_AKKKK, Custom Footprints:SOT-753, symbol Custom_parts:D_Zener_x4_ACom_AKKKK
- removed J6: Conn_01x05_Male, Custom Footprints:Ref_only, symbol Custom_parts:Conn_01x05_Male
- removed J9: Conn_01x04_Male, Custom Footprints:Ref_only, symbol Custom_parts:Conn_01x04_Male
- removed RN2: 220, Custom Footprints:Bourns_16-SOIC_8x_r-pack, symbol Device:R_Pack08_Split
- removed RV9: R_POT_SPST, Custom Footprints:P091S-FC20BR10K, symbol Custom_parts:R_POT_SPST
- removed SW1: G13JVCF, Custom Footprints:G13JVCF_or_GW12LJVCF, symbol Switch:SW_NKK_GW12LJPCF
- removed U1: S20V18F122V_DC, Custom Footprints:S18V20F12_12V_DC, symbol Custom_parts:S18V20F12_12V_DC
- added C4: 47uF, Capacitor_SMD:C_1206_3216Metric, symbol Device:C_Small
- added J10: Conn_01x08_Female, Custom Footprints:Ref_only, symbol Custom_parts:Conn_01x08_Female
- added J4: Conn_01x05_Female, Custom Footprints:Ref_only, symbol Custom_parts:Conn_01x05_Female
- added J6: Conn_01x03_Male, Custom Footprints:Ref_only, symbol Custom_parts:Conn_01x03_Male
- added J8, J9: Conn_01x03_Female, Custom Footprints:Ref_only, symbol Custom_parts:Conn_01x03_Female
- added JP2: SolderJumper_2_Open, Jumper:SolderJumper-2_P1.3mm_Open_TrianglePad1.0x1.5mm, symbol Jumper:SolderJumper_2_Open
- added RN2: 150, Resistor_SMD:R_Array_Convex_4x1206, symbol Device:R_Pack04_Split
- added RN4: R_Pack04, Resistor_SMD:R_Array_Convex_4x1206, symbol Device:R_Pack04
- added RV3: R_POT, Custom Footprints:Pot_with_header, symbol Device:R_POT
- added SW1: SW_SPDT, Custom Footprints:1x5_header_SSM-105-L-SV-BE-LC, symbol Switch:SW_SPDT
- added SW2, SW3, SW4, SW5: Pushbutton_with_LED_-_ELUMOATHQ3C12, Custom Footprints:Pushbutton_LED-ELUMOATHQ3C12, symbol Custom_parts:Pushbutton_with_LED_-_ELUMOATHQ3C12
- added U1: 12V boost, Custom Footprints:12V_DC-DC_with_header_2117, symbol Regulator_Switching:R-78B1.2-2.0
- BZ1: footprint Custom Footprints:XDCR_CPT-2016-75-SMT-TR -> Custom Footprints:SMT-0940-T-3V-R_9x9_alarm; Manufacturer CUI Devices -> PUI Audio, Inc.; Part # CPT-2016-75-SMT-TR -> SMT-0940-T-3V-R
- C1, C2, C3: value 14000uF -> 7500uF
- J2, JP1: footprint Connector_Wire:SolderWire-2.5sqmm_1x02_P7.2mm_D2.4mm_OD3.6mm -> Custom Footprints:Wire_Pad
- M1: footprint Connector_Wire:SolderWire-0.25sqmm_1x04_P4.2mm_D0.65mm_OD1.7mm -> Custom Footprints:4-pin_fan_SMD; Manufacturer (none) -> Samtec Inc.; Part # (none) -> TSM-104-02-L-SV
- RN3: footprint Custom Footprints:Bourns_16-SOIC_8x_r-pack -> Custom Footprints:2506_8x_R-pack; Manufacturer Bourns Inc. -> CTS Resistor Products; Part # 4816P-T01-472LF -> 742C163472JP
- U3: footprint Custom Footprints:DPBW06F-05 -> Custom Footprints:DPBW06F-05_with_header
Connections:
- net labels added: Button1, Button2, Button3, Button4, LED1, LED2, LED3, LED4, Relay1, Relay2, Relay3, Relay4, SCL0, SDA0
- net labels removed: 5V-analog, LCD_CS, LCD_reset, Pushbutton_switch, external_analog_2, external_analog_3, external_analog_4
- no-connect marks 47 -> 53
Other:
- note added: "Add SMD 4-pin connector for 4 pin fan\n-Include Fan guard\n\nSwitch supply so smaller boost supply\n"
- note added: "Boost - Vin (3V - 12V) to 12V DC"
- note added: "LED bypass capacitors and connectors\nFor high current supplies use an in-line\ncapacitor with the power supply such as:\nUnited Chemi-Con E32D500HPN104MDA5M"
- note added: "Manual/Auto toggle switch"
- note added: "Pot to adjust LED intensity"
- note removed: "4-channel external analog input with 5.6V zener clamp\nAbsolute max voltage: +11V/-6V"
- note removed: "Add fan and molex connector\n-Put molex near RN3 (since it also needs Vin) and U16 (since this is the source for the fan PWM)\n-Include Fan guard\n\nSwith thermistor R-pack to x4\n\nAdd pushbutton with LED\n\nSwith 150 ohm R-pack to 5-8x to accomodate pushbutton LED"
- note removed: "Can replace\nwith GW12LJVCF"
- note removed: "Header pins\nto connect\n12V SEPIC \nDC-DC \nconverter"
- note removed: "Internal 4-channel 12-bit DAC AWG"
- note removed: "LED bypass capacitors and connectors"
- note removed: "Manual/Auto toggle switch with indicator LED"
- note removed: "Maximum 25V Vin with \n1k impedance on Isense"
- note removed: "SEPIC - Vin (3V - 30V) to 12V DC"
- moved on the sheet: U2, U7, U8, U9

Commit message: More layout work - only one isolated ground island
Parts:
- removed C18: 2.2uF, Custom Footprints:0508_Capacitor, symbol Device:C_Small
- removed JP2: SolderJumper_2_Open, Jumper:SolderJumper-2_P1.3mm_Open_TrianglePad1.0x1.5mm, symbol Jumper:SolderJumper_2_Open
- added C9: 2200pF, Capacitor_SMD:C_0603_1608Metric, symbol Device:C_Small
Connections:
- net GND: now also R1.2, R3.2, R4.2, R5.2, C9.1; no longer R1.1, R3.1, R4.1, R5.1
- net Isense: now also R1.1, R3.1, R4.1, R5.1; no longer R1.2, R3.2, R4.2, R5.2
- net LED1: now also RN2.4 (R4.1); no longer RN2.1 (R1.1)
- net LED2: now also RN2.3 (R3.1); no longer RN2.2 (R2.1)
- net LED3: now also RN2.2 (R2.1); no longer RN2.3 (R3.1)
- net LED4: now also RN2.1 (R1.1); no longer RN2.4 (R4.1)
- net MOSFET_temp: no longer J7.~, U14.43 (16_A2_SCL0_TOUCH)
- net at RN3.5 (R5.1), U6.5 (EN), U6.6 (VDD): now also C9.2
- net at SW2.5 (A): now also RN2.5 (R4.2); no longer RN2.8 (R1.2)
- net at SW3.5 (A): now also RN2.6 (R3.2); no longer RN2.7 (R2.2)
- net at SW4.5 (A): now also RN2.7 (R2.2); no longer RN2.6 (R3.2)
- net at SW5.5 (A): now also RN2.8 (R1.2); no longer RN2.5 (R4.2)
- new net: J7.~, U14.43 (16_A2_SCL0_TOUCH)
Other:
- note added: "Use smaller LDOs - especially lower dropout on 10V rail\nUse lower wattage (smaller) resistor on 1.8V rail\nAdd RC filter to 12V input to 10V LDO\nRemove inductor and use same rail for 12V to 10V LDO?\nSee if there is a bigger zener set for D6 or split to 2 parts"
- note removed: "Add SMD 4-pin connector for 4 pin fan\n-Include Fan guard\n\nSwitch supply so smaller boost supply\n"
- moved on the sheet: RN2A, RN2B, RN2C, RN2D
Changed lines of the file:
@@
 F 5 "TKH45P5R00FE-TR" H 11350 8150 50  0001 C CNN "Part #"
 	1    11350 8150
-	1    0    0    1
+	-1   0    0    -1
 $EndComp
 Text Notes 10950 6800 0    59   ~ 0
@@
 Wire Wire Line
 	5550 2200 5650 2200
-Connection ~ 5400 6850
 $Comp
 L Custom_parts:8P8C_Shielded_x4 J3
@@
 Text Label 13100 1600 0    50   ~ 0
 LED_pot
-Text Label 13100 2000 0    50   ~ 0
+Text Label 15050 2750 0    50   ~ 0
 MOSFET_temp
 Text Label 3200 9050 0    50   ~ 0
@@
 Text Label 10800 3100 2    50   ~ 0
 External_5V_PWM2
-$Comp
-L Device:C_Small C18
-U 1 1 5F422B07
-P 5500 6850
-F 0 "C18" V 5700 6800 50  0000 L CNN
-F 1 "2.2uF" V 5600 6800 50  0000 L CNN
-F 2 "Custom Footprints:0508_Capacitor" H 5500 6850 50  0001 C CNN
-F 3 "https://ds.yuden.co.jp/TYCOMPAS/ut/detail?pn=TWK212B7225MD-T%20&u=M" H 5500 6850 50  0001 C CNN
-F 4 "Taiyo Yuden" H 5500 6850 50  0001 C CNN "Manufacturer"
-F 5 "TWK212B7225MD-T" H 5500 6850 50  0001 C CNN "Part #"
-	1    5500 6850
-	0    1    1    0
-$EndComp
 Wire Wire Line
 	4650 6900 3900 6900
@@
 Text Label 13100 2800 0    50   ~ 0
 Pushbutton_LED
-Text Notes 2950 -1300 0    157  ~ 0
-Add SMD 4-pin connector for 4 pin fan\n-Include Fan guard\n\nSwitch supply so smaller boost supply\n
 Connection ~ 11350 8050
 Wire Wire Line
@@
 F 5 "TKH45P5R00FE-TR" H 11550 8150 50  0001 C CNN "Part #"
 	1    11550 8150
-	1    0    0    1
+	-1   0    0    -1
 $EndComp
 $Comp
@@
 F 5 "TKH45P5R00FE-TR" H 11750 8150 50  0001 C CNN "Part #"
 	1    11750 8150
-	1    0    0    1
+	-1   0    0    -1
 $EndComp
 $Comp
@@
 F 5 "TKH45P5R00FE-TR" H 11950 8150 50  0001 C CNN "Part #"
 	1    11950 8150
-	1    0    0    1
-$EndComp
-Wire Wire Line
-	11350 8050 11550 8050
-Connection ~ 11550 8050
-Wire Wire Line
-	11550 8050 11750 8050
-Connection ~ 11750 8050
-Wire Wire Line
-	11750 8050 11950 8050
-Wire Wire Line
-	11950 8250 11750 8250
-Connection ~ 11350 8250
-Connection ~ 11550 8250
-Wire Wire Line
-	11550 8250 11350 8250
-Connection ~ 11750 8250
-Wire Wire Line
-	11750 8250 11550 8250
+	-1   0    0    -1
+$EndComp
 Wire Notes Line
 	500  6000 8750 6000
@@
 	1    0    0    -1
 $EndComp
-Wire Wire Line
-	1350 1650 1850 1650
-Wire Wire Line
-	2600 1650 2750 1650
 $Comp
 L power:GND #PWR0121
@@
 Text Label 2650 1000 2    50   ~ 0
 12V
-$Comp
-L Jumper:SolderJumper_2_Open JP2
-U 1 1 5F822B93
-P 2300 2350
-F 0 "JP2" H 2300 2555 50  0000 C CNN
-F 1 "SolderJumper_2_Open" H 2300 2464 50  0000 C CNN
-F 2 "Jumper:SolderJumper-2_P1.3mm_Open_TrianglePad1.0x1.5mm" H 2300 2350 50  0001 C CNN
-F 3 "~" H 2300 2350 50  0001 C CNN
-	1    2300 2350
-	1    0    0    -1
-$EndComp
-Wire Wire Line
-	2150 2350 1850 2350
-Wire Wire Line
-	1850 2350 1850 1650
-Connection ~ 1850 1650
-Wire Wire Line
-	1850 1650 2000 1650
-Wire Wire Line
-	2450 2350 2750 2350
-Wire Wire Line
-	2750 2350 2750 1650
-Connection ~ 2750 1650
-Wire Wire Line
-	2750 1650 2850 1650
 $Comp
 L Custom_parts:Conn_01x08_Female J10
@@
 L Device:R_Pack04_Split RN2
 U 1 1 5F9E09BB
+P 9800 5050
+F 0 "RN2" V 9900 5050 50  0000 C CNN
+F 1 "150" V 9800 5050 50  0000 C CNN
+F 2 "Resistor_SMD:R_Array_Convex_4x1206" V 10075 5050 50  0001 C CNN
+F 3 "https://industrial.panasonic.com/cdbs/www-data/pdf/AOC0000/AOC0000C14.pdf" H 9800 5050 50  0001 C CNN
+F 4 "Panasonic Electronic Components" V 9800 5050 50  0001 C CNN "Manufacturer"
+F 5 "EXB-38V151JV" V 9800 5050 50  0001 C CNN "Part #"
+	1    9800 5050
+	0    -1   -1   0
+$EndComp
+$Comp
+L Device:R_Pack04_Split RN2
+U 2 1 5F9E5ED4
+P 9800 4300
+F 0 "RN2" V 9900 4300 50  0000 C CNN
+F 1 "150" V 9800 4300 50  0000 C CNN
+F 2 "Resistor_SMD:R_Array_Convex_4x1206" V 10075 4300 50  0001 C CNN
+F 3 "https://industrial.panasonic.com/cdbs/www-data/pdf/AOC0000/AOC0000C14.pdf" H 9800 4300 50  0001 C CNN
+F 4 "Panasonic Electronic Components" V 9800 4300 50  0001 C CNN "Manufacturer"
+F 5 "EXB-38V151JV" V 9800 4300 50  0001 C CNN "Part #"
+	2    9800 4300
+	0    -1   -1   0
+$EndComp
+$Comp
+L Device:R_Pack04_Split RN2
+U 3 1 5F9E7B6F
+P 8200 5050
+F 0 "RN2" V 8300 5050 50  0000 C CNN
+F 1 "150" V 8200 5050 50  0000 C CNN
+F 2 "Resistor_SMD:R_Array_Convex_4x1206" V 8475 5050 50  0001 C CNN
+F 3 "https://industrial.panasonic.com/cdbs/www-data/pdf/AOC0000/AOC0000C14.pdf" H 8200 5050 50  0001 C CNN
+F 4 "Panasonic Electronic Components" V 8200 5050 50  0001 C CNN "Manufacturer"
+F 5 "EXB-38V151JV" V 8200 5050 50  0001 C CNN "Part #"
+	3    8200 5050
+	0    -1   -1   0
+$EndComp
+$Comp
+L Device:R_Pack04_Split RN2
+U 4 1 5F9E8C0F
 P 8200 4300
 F 0 "RN2" V 8300 4300 50  0000 C CNN
@@
 F 4 "Panasonic Electronic Components" V 8200 4300 50  0001 C CNN "Manufacturer"
 F 5 "EXB-38V151JV" V 8200 4300 50  0001 C CNN "Part #"
-	1    8200 4300
-	0    -1   -1   0
-$EndComp
-$Comp
-L Device:R_Pack04_Split RN2
-U 2 1 5F9E5ED4
-P 8200 5050
-F 0 "RN2" V 8300 5050 50  0000 C CNN
-F 1 "150" V 8200 5050 50  0000 C CNN
-F 2 "Resistor_SMD:R_Array_Convex_4x1206" V 8475 5050 50  0001 C CNN
-F 3 "https://industrial.panasonic.com/cdbs/www-data/pdf/AOC0000/AOC0000C14.pdf" H 8200 5050 50  0001 C CNN
-F 4 "Panasonic Electronic Components" V 8200 5050 50  0001 C CNN "Manufacturer"
-F 5 "EXB-38V151JV" V 8200 5050 50  0001 C CNN "Part #"
-	2    8200 5050
-	0    -1   -1   0
-$EndComp
-$Comp
-L Device:R_Pack04_Split RN2
-U 3 1 5F9E7B6F
-P 9800 4300
-F 0 "RN2" V 9900 4300 50  0000 C CNN
-F 1 "150" V 9800 4300 50  0000 C CNN
-F 2 "Resistor_SMD:R_Array_Convex_4x1206" V 10075 4300 50  0001 C CNN
-F 3 "https://industrial.panasonic.com/cdbs/www-data/pdf/AOC0000/AOC0000C14.pdf" H 9800 4300 50  0001 C CNN
-F 4 "Panasonic Electronic Components" V 9800 4300 50  0001 C CNN "Manufacturer"
-F 5 "EXB-38V151JV" V 9800 4300 50  0001 C CNN "Part #"
-	3    9800 4300
-	0    -1   -1   0
-$EndComp
-$Comp
-L Device:R_Pack04_Split RN2
-U 4 1 5F9E8C0F
-P 9800 5050
-F 0 "RN2" V 9900 5050 50  0000 C CNN
-F 1 "150" V 9800 5050 50  0000 C CNN
-F 2 "Resistor_SMD:R_Array_Convex_4x1206" V 10075 5050 50  0001 C CNN
-F 3 "https://industrial.panasonic.com/cdbs/www-data/pdf/AOC0000/AOC0000C14.pdf" H 9800 5050 50  0001 C CNN
-F 4 "Panasonic Electronic Components" V 9800 5050 50  0001 C CNN "Manufacturer"
-F 5 "EXB-38V151JV" V 9800 5050 50  0001 C CNN "Part #"
-	4    9800 5050
+	4    8200 4300
 	0    -1   -1   0
 $EndComp
@@
 	1    0    0    -1
 $EndComp
+Text Notes 4550 -50  0    118  ~ 0
+Use smaller LDOs - especially lower dropout on 10V rail\nUse lower wattage (smaller) resistor on 1.8V rail\nAdd RC filter to 12V input to 10V LDO\nRemove inductor and use same rail for 12V to 10V LDO?\nSee if there is a bigger zener set for D6 or split to 2 parts
+Wire Wire Line
+	1350 1650 2000 1650
+Wire Wire Line
+	2600 1650 2850 1650
+$Comp
+L Device:C_Small C9
+U 1 1 5F565AC5
+P 5500 6850
+F 0 "C9" V 5400 6850 50  0000 C CNN
+F 1 "2200pF" V 5300 6850 50  0000 C CNN
+F 2 "Capacitor_SMD:C_0603_1608Metric" H 5500 6850 50  0001 C CNN
+F 3 "https://api.kemet.com/component-edge/download/datasheet/C0603C222K1RACTU.pdf" H 5500 6850 50  0001 C CNN
+F 4 "KEMET" H 5500 6850 50  0001 C CNN "Manufacturer"
+F 5 "C0603C222K1RACTU" H 5500 6850 50  0001 C CNN "Part #"
+	1    5500 6850
+	0    1    -1   0
+$EndComp
+Connection ~ 5400 6850
+Connection ~ 11350 8250
+Wire Wire Line
+	11350 8050 11550 8050
+Wire Wire Line
+	11350 8250 11550 8250
+Connection ~ 11550 8050
+Connection ~ 11550 8250
+Wire Wire Line
+	11550 8050 11750 8050
+Wire Wire Line
+	11550 8250 11750 8250
+Connection ~ 11750 8050
+Wire Wire Line
+	11750 8050 11950 8050
+Connection ~ 11750 8250
+Wire Wire Line
+	11750 8250 11950 8250
 $EndSCHEMATC
