File: KiCAD/Four Channel MHz LED Driver/Four Channel MHz LED Driver - high current.kicad_pcb (KiCad board)
At the start: 2 copper layers, 100 x 126 mm, 85 parts, among them J10 Conn_01x24_Female, J2 Conn_01x02_Female, J3 8P8C_Shielded_x4, J4 Conn_01x03_Male, J5 Conn_01x03_Female, J6 Conn_01x08_Female, J7 Conn_01x03_Female, J8 Conn_01x05_Female, J9 Conn_01x24_Female, M1 Fan_4pin, Q1 SUM70060E, SW1 Pushbutton_with_LED, SW2 Pushbutton_with_LED, SW3 Pushbutton_with_LED, SW4 Pushbutton_with_LED, SW5 SW_SPDT, U1 12V boost, U12 Teensy3.6, U2 SN74LV4T125PWR, U3 DPBW06F-05, U4 TMUX1204DGSR, U5 HTSOP-J8_ROM, U6 ADP7182AUJZ-1.8-R7, U7 LT6200CS8-10

Commit message: Driver updates
Parts:
- RN3: footprint Custom Footprints:2506_modified_concave_8x_R-pack -> Custom Footprints:1506-EXB-2HV472JV-for_2_oz_pour
- U5: value HTSOP-J8_ROM -> BDJ0GA5WEFJ-E2
- moved JP1 3.25 mm to (79.2, 122.7)
- moved TH2 0.75 mm to (143.3, 121.3)
- moved RN3 0.26 mm to (135.3, 74.9), turned to 270 degrees
Routing:
- net /MOSFET_temp: track 157.6 -> 159.9 mm
- net /Resistor_temp: track 98.5 -> 100.1 mm
- net /A-D_input_4: track 33.1 -> 34.2 mm
- net /External_thermistor: track 76.4 -> 77.3 mm
- net Net-(J3-Pad29): track 15.1 -> 15.8 mm
- net GND: track 873.7 -> 874.4 mm
- net Net-(J3-Pad31): track 13.7 -> 14.3 mm
- net /A-D_input_3: track 37.2 -> 37.8 mm
